File: Sequencer.kicad_pcb (KiCad board)
At the start: 2 copper layers, 0 parts

Commit message: Fixed some footprints and models.
Parts:
- added C1: 10u, Capacitor_SMD:CP_Elec_4x5.8, F.Cu at (198.9, 119.2)
- added C10: 47n, Capacitor_SMD:C_0603_1608Metric, F.Cu at (147.3, 78.9)
- added C11: 47n, Capacitor_SMD:C_0603_1608Metric, F.Cu at (156.3, 80.4)
- added C12: 47n, Capacitor_SMD:C_0603_1608Metric, F.Cu at (162.3, 78.3)
- added C13: 47n, Capacitor_SMD:C_0603_1608Metric, F.Cu at (162.3, 79.8)
- added C14: 47n, Capacitor_SMD:C_0603_1608Metric, F.Cu at (165.3, 76.8)
- added C15: 47n, Capacitor_SMD:C_0603_1608Metric, F.Cu at (165.3, 78.3)
- added C16: 47n, Capacitor_SMD:C_0603_1608Metric, F.Cu at (168.3, 75.3)
- added C17: 100p, Capacitor_SMD:C_0603_1608Metric, F.Cu at (165.3, 79.8)
- added C18: 100p, Capacitor_SMD:C_0603_1608Metric, F.Cu at (168.3, 76.8)
- added C19: 100p, Capacitor_SMD:C_0603_1608Metric, F.Cu at (162.3, 82.9)
- added C2: 10u, Capacitor_SMD:CP_Elec_4x5.8, F.Cu at (209.4, 114.3)
- added C20: 100p, Capacitor_SMD:C_0603_1608Metric, F.Cu at (173.3, 73.8)
- added C21: 100n, Capacitor_SMD:C_0603_1608Metric, F.Cu at (170.2, 73.8)
- added C22: 100n, Capacitor_SMD:C_0603_1608Metric, F.Cu at (147.3, 82.9)
- added C23: 47n, Capacitor_SMD:C_0603_1608Metric, F.Cu at (94.9, 144.4)
- added C24: 47n, Capacitor_SMD:C_0603_1608Metric, F.Cu at (104.0, 143.4)
- added C25: 47n, Capacitor_SMD:C_0603_1608Metric, F.Cu at (113.0, 139.8)
- added C26: 47n, Capacitor_SMD:C_0603_1608Metric, F.Cu at (107.0, 141.9)
- added C27: 47n, Capacitor_SMD:C_0603_1608Metric, F.Cu at (104.0, 141.9)
- added C28: 47n, Capacitor_SMD:C_0603_1608Metric, F.Cu at (101.0, 141.9)
- added C29: 47n, Capacitor_SMD:C_0603_1608Metric, F.Cu at (97.9, 142.9)
- added C3: 100n, Capacitor_SMD:C_0603_1608Metric, F.Cu at (207.1, 122.4)
- added C30: 47n, Capacitor_SMD:C_0603_1608Metric, F.Cu at (97.9, 141.4)
- added C31: 100p, Capacitor_SMD:C_0603_1608Metric, F.Cu at (94.9, 141.9)
- added C32: 100p, Capacitor_SMD:C_0603_1608Metric, F.Cu at (107.0, 140.4)
- added C33: 100p, Capacitor_SMD:C_0603_1608Metric, F.Cu at (104.0, 140.4)
- added C34: 100p, Capacitor_SMD:C_0603_1608Metric, F.Cu at (101.0, 140.4)
- added C35: 100n, Capacitor_SMD:C_0603_1608Metric, F.Cu at (107.0, 138.9)
- added C36: 100n, Capacitor_SMD:C_0603_1608Metric, F.Cu at (104.0, 138.9)
- added C37: 100n, Capacitor_SMD:C_0603_1608Metric, F.Cu at (94.9, 77.9)
- added C38: 100n, Capacitor_SMD:C_0603_1608Metric, F.Cu at (96.5, 80.9)
- added C39: 100n, Capacitor_SMD:C_0603_1608Metric, F.Cu at (99.5, 77.9)
- added C4: 100n, Capacitor_SMD:C_0603_1608Metric, F.Cu at (200.0, 125.1)
- added C40: 100n, Capacitor_SMD:C_0603_1608Metric, F.Cu at (102.5, 74.9)
- added C41: 470p, Capacitor_SMD:C_0603_1608Metric, F.Cu at (93.5, 84.2)
- added C42: 470p, Capacitor_SMD:C_0603_1608Metric, F.Cu at (90.5, 85.8)
- added C43: 100n, Capacitor_SMD:C_0603_1608Metric, F.Cu at (123.3, 91.2)
- added C44: 100n, Capacitor_SMD:C_0603_1608Metric, F.Cu at (97.9, 105.7)
- added C45: 100n, Capacitor_SMD:C_0603_1608Metric, F.Cu at (105.5, 105.7)
- added C46: 100n, Capacitor_SMD:C_0603_1608Metric, F.Cu at (94.9, 108.7)
- added C47: 470p, Capacitor_SMD:C_0603_1608Metric, F.Cu at (87.5, 115.0)
- added C48: 470p, Capacitor_SMD:C_0603_1608Metric, F.Cu at (94.9, 107.2)
- added C5: 10u, Capacitor_SMD:CP_Elec_4x5.8, F.Cu at (205.6, 119.2)
- added C6: 100n, Capacitor_SMD:C_0603_1608Metric, F.Cu at (142.8, 98.3)
- added C7: 100n, Capacitor_SMD:C_0603_1608Metric, F.Cu at (139.8, 99.8)
- added C8: 100n, Capacitor_SMD:C_0603_1608Metric, F.Cu at (145.8, 98.3)
- added C9: 47n, Capacitor_SMD:C_0603_1608Metric, F.Cu at (150.3, 75.9)
- added D1: DFLR1400-7, Diode_SMD:D_PowerDI-123, F.Cu at (211.5, 118.0)
- added D2: DFLR1400-7, Diode_SMD:D_PowerDI-123, F.Cu at (203.1, 123.0)
- added D3: LED, LED_SMD:LED_1206_3216Metric_Castellated, F.Cu at (198.0, 122.8)
- added D4: LM4040DBZ-10, Package_TO_SOT_SMD:SOT-23, F.Cu at (140.0, 108.6)
- added J-Inv1: AudioJack2_Ground_Switch, Local:PJ398SM, F.Cu at (176.4, 65.8)
- added J-Inv10: AudioJack2_Ground_Switch, Local:PJ398SM, F.Cu at (136.6, 127.3)
- added J-Inv11: AudioJack2_Ground_Switch, Local:PJ398SM, F.Cu at (175.8, 93.0)
- added J-Inv12: AudioJack2_Ground_Switch, Local:PJ398SM, F.Cu at (217.7, 65.8)
- added J-Inv13: AudioJack2_Ground_Switch, Local:PJ398SM, F.Cu at (117.3, 65.8)
- added J-Inv14: AudioJack2_Ground_Switch, Local:PJ398SM, F.Cu at (117.3, 79.1)
- added J-Inv15: AudioJack2_Ground_Switch, Local:PJ398SM, F.Cu at (117.3, 96.5)
- added J-Inv16: AudioJack2_Ground_Switch, Local:PJ398SM, F.Cu at (117.3, 109.9)
- added J-Inv2: AudioJack2_Ground_Switch, Local:PJ398SM, F.Cu at (167.3, 65.8)
- added J-Inv3: AudioJack2_Ground_Switch, Local:PJ398SM, F.Cu at (189.0, 65.8)
- added J-Inv4: AudioJack2_Ground_Switch, Local:PJ398SM, F.Cu at (165.4, 112.9)
- added J-Inv5: AudioJack2_Ground_Switch, Local:PJ398SM, F.Cu at (204.6, 83.2)
- added J-Inv6: AudioJack2_Ground_Switch, Local:PJ398SM, F.Cu at (115.0, 127.3)
- added J-Inv7: AudioJack2_Ground_Switch, Local:PJ398SM, F.Cu at (124.1, 127.3)
- added J-Inv8: AudioJack2_Ground_Switch, Local:PJ398SM, F.Cu at (165.4, 130.2)
- added J-Inv9: AudioJack2_Ground_Switch, Local:PJ398SM, F.Cu at (204.6, 100.6)
- added J1: Conn_02x05_Odd_Even, Connector_PinHeader_2.54mm:PinHeader_2x05_P2.54mm_Vertical, F.Cu at (191.1, 113.7)
- added J2: Conn_02x03_Odd_Even, Connector_PinHeader_2.54mm:PinHeader_2x03_P2.54mm_Vertical, F.Cu at (160.3, 88.7)
- added J3: Conn_01x03, Connector_PinHeader_2.54mm:PinHeader_1x03_P2.54mm_Vertical, F.Cu at (150.8, 96.3)
- added Q1: BC847, Package_TO_SOT_SMD:SOT-23, F.Cu at (195.3, 61.5)
- added Q2: BC847, Package_TO_SOT_SMD:SOT-23, F.Cu at (142.9, 123.0)
- added Q3: BC847, Package_TO_SOT_SMD:SOT-23, F.Cu at (182.1, 88.7)
- added Q4: BC847, Package_TO_SOT_SMD:SOT-23, F.Cu at (224.0, 61.5)
- added R1: 330, Resistor_SMD:R_0603_1608Metric, F.Cu at (197.0, 124.7)
- added R10: 470, Resistor_SMD:R_0603_1608Metric, F.Cu at (165.3, 75.3)
- added R11: 68k, Resistor_SMD:R_0603_1608Metric, F.Cu at (162.3, 76.8)
- added R12: 68k, Resistor_SMD:R_0603_1608Metric, F.Cu at (150.3, 78.3)
- added R13: 33k, Resistor_SMD:R_0603_1608Metric, F.Cu at (153.3, 77.4)
- added R14: 33k, Resistor_SMD:R_0603_1608Metric, F.Cu at (156.3, 77.4)
- added R15: 68k, Resistor_SMD:R_0603_1608Metric, F.Cu at (159.3, 77.4)
- added R16: 68k, Resistor_SMD:R_0603_1608Metric, F.Cu at (153.3, 78.9)
- added R17: 470, Resistor_SMD:R_0603_1608Metric, F.Cu at (156.3, 78.9)
- added R18: 1k5, Resistor_SMD:R_0603_1608Metric, F.Cu at (159.3, 78.9)
- added R19: 470, Resistor_SMD:R_0603_1608Metric, F.Cu at (147.3, 80.4)
- added R2: 10k, Resistor_SMD:R_0603_1608Metric, F.Cu at (139.8, 98.3)
- added R20: 1k5, Resistor_SMD:R_0603_1608Metric, F.Cu at (150.3, 79.8)
- added R21: 2k2, Resistor_SMD:R_0603_1608Metric, F.Cu at (156.3, 81.9)
- added R22: 2k2, Resistor_SMD:R_0603_1608Metric, F.Cu at (153.3, 80.4)
- added R23: 2k2, Resistor_SMD:R_0603_1608Metric, F.Cu at (162.3, 81.3)
- added R24: 2k2, Resistor_SMD:R_0603_1608Metric, F.Cu at (159.3, 80.4)
- added R25: 68k, Resistor_SMD:R_0603_1608Metric, F.Cu at (167.2, 73.8)
- added R26: 68k, Resistor_SMD:R_0603_1608Metric, F.Cu at (147.3, 77.4)
- added R27: 33k, Resistor_SMD:R_0603_1608Metric, F.Cu at (150.3, 74.3)
- added R28: 33k, Resistor_SMD:R_0603_1608Metric, F.Cu at (164.2, 73.8)
- added R29: 68k, Resistor_SMD:R_0603_1608Metric, F.Cu at (150.3, 81.3)
- added R3: 470, Resistor_SMD:R_0603_1608Metric, F.Cu at (153.3, 74.3)
- added R30: 68k, Resistor_SMD:R_0603_1608Metric, F.Cu at (159.3, 81.9)
- added R31: 100k, Resistor_SMD:R_0603_1608Metric, F.Cu at (150.3, 82.9)
- added R32: 100k, Resistor_SMD:R_0603_1608Metric, F.Cu at (153.3, 81.9)
- added R33: 1k, Resistor_SMD:R_0603_1608Metric, F.Cu at (147.3, 75.9)
- added R34: 1k, Resistor_SMD:R_0603_1608Metric, F.Cu at (147.3, 74.3)
- added R35: 100k, Resistor_SMD:R_0603_1608Metric, F.Cu at (198.5, 60.4)
- added R36: 10k, Resistor_SMD:R_0603_1608Metric, F.Cu at (195.0, 64.0)
- added R37: 1k, Resistor_SMD:R_0603_1608Metric, F.Cu at (175.3, 107.5)
- added R38: 1k, Resistor_SMD:R_0603_1608Metric, F.Cu at (214.5, 77.9)
- added R39: 470, Resistor_SMD:R_0603_1608Metric, F.Cu at (107.0, 143.4)
- added R4: 470, Resistor_SMD:R_0603_1608Metric, F.Cu at (156.3, 74.3)
- added R40: 470, Resistor_SMD:R_0603_1608Metric, F.Cu at (101.0, 143.4)
- added R41: 470, Resistor_SMD:R_0603_1608Metric, F.Cu at (116.0, 136.8)
- added R42: 470, Resistor_SMD:R_0603_1608Metric, F.Cu at (101.0, 138.9)
- added R43: 470, Resistor_SMD:R_0603_1608Metric, F.Cu at (97.9, 139.8)
- added R44: 470, Resistor_SMD:R_0603_1608Metric, F.Cu at (94.9, 137.4)
- added R45: 470, Resistor_SMD:R_0603_1608Metric, F.Cu at (94.9, 135.9)
- added R46: 470, Resistor_SMD:R_0603_1608Metric, F.Cu at (97.9, 144.4)
- added R47: 68k, Resistor_SMD:R_0603_1608Metric, F.Cu at (110.0, 144.4)
- added R48: 68k, Resistor_SMD:R_0603_1608Metric, F.Cu at (113.0, 141.4)
- added R49: 33k, Resistor_SMD:R_0603_1608Metric, F.Cu at (116.0, 138.3)
- added R5: 470, Resistor_SMD:R_0603_1608Metric, F.Cu at (159.3, 74.3)
- added R50: 33k, Resistor_SMD:R_0603_1608Metric, F.Cu at (120.9, 135.3)
- added R51: 68k, Resistor_SMD:R_0603_1608Metric, F.Cu at (110.0, 142.9)
- added R52: 68k, Resistor_SMD:R_0603_1608Metric, F.Cu at (117.9, 135.3)
- added R53: 470, Resistor_SMD:R_0603_1608Metric, F.Cu at (113.0, 138.3)
- added R54: 1k5, Resistor_SMD:R_0603_1608Metric, F.Cu at (110.0, 141.4)
- added R55: 470, Resistor_SMD:R_0603_1608Metric, F.Cu at (110.0, 139.8)
- added R56: 1k5, Resistor_SMD:R_0603_1608Metric, F.Cu at (114.9, 135.3)
- added R57: 2k2, Resistor_SMD:R_0603_1608Metric, F.Cu at (94.9, 138.9)
- added R58: 2k2, Resistor_SMD:R_0603_1608Metric, F.Cu at (97.9, 135.9)
- added R59: 2k2, Resistor_SMD:R_0603_1608Metric, F.Cu at (111.9, 135.3)
- added R6: 470, Resistor_SMD:R_0603_1608Metric, F.Cu at (153.3, 75.9)
- added R60: 2k2, Resistor_SMD:R_0603_1608Metric, F.Cu at (97.9, 137.4)
- added R61: 68k, Resistor_SMD:R_0603_1608Metric, F.Cu at (94.9, 140.4)
- added R62: 68k, Resistor_SMD:R_0603_1608Metric, F.Cu at (101.0, 135.9)
- added R63: 33k, Resistor_SMD:R_0603_1608Metric, F.Cu at (104.0, 135.9)
- added R64: 33k, Resistor_SMD:R_0603_1608Metric, F.Cu at (107.0, 135.9)
- added R65: 68k, Resistor_SMD:R_0603_1608Metric, F.Cu at (101.0, 137.4)
- added R66: 68k, Resistor_SMD:R_0603_1608Metric, F.Cu at (104.0, 137.4)
- added R67: 100k, Resistor_SMD:R_0603_1608Metric, F.Cu at (107.0, 137.4)
- added R68: 100k, Resistor_SMD:R_0603_1608Metric, F.Cu at (110.0, 136.8)
- added R69: 1k, Resistor_SMD:R_0603_1608Metric, F.Cu at (113.0, 136.8)
- added R7: 470, Resistor_SMD:R_0603_1608Metric, F.Cu at (156.3, 75.9)
- added R70: 1k, Resistor_SMD:R_0603_1608Metric, F.Cu at (110.0, 138.3)
- added R71: 1k, Resistor_SMD:R_0603_1608Metric, F.Cu at (175.3, 124.9)
- added R72: 1k, Resistor_SMD:R_0603_1608Metric, F.Cu at (214.5, 95.3)
- added R73: 100k, Resistor_SMD:R_0603_1608Metric, F.Cu at (142.7, 125.5)
- added R74: 10k, Resistor_SMD:R_0603_1608Metric, F.Cu at (146.2, 122.0)
- added R75: 100k, Resistor_SMD:R_0603_1608Metric, F.Cu at (185.4, 87.7)
- added R76: 10k, Resistor_SMD:R_0603_1608Metric, F.Cu at (181.9, 91.2)
- added R77: 100k, Resistor_SMD:R_0603_1608Metric, F.Cu at (227.2, 60.4)
- added R78: 10k, Resistor_SMD:R_0603_1608Metric, F.Cu at (223.8, 64.0)
- added R79: 2k2, Resistor_SMD:R_0603_1608Metric, F.Cu at (143.3, 107.5)
- added R8: 470, Resistor_SMD:R_0603_1608Metric, F.Cu at (159.3, 75.9)
- added R80: 100k, Resistor_SMD:R_0603_1608Metric, F.Cu at (97.9, 76.4)
- added R81: 200k, Resistor_SMD:R_0603_1608Metric, F.Cu at (94.9, 79.4)
- added R82: 100k, Resistor_SMD:R_0603_1608Metric, F.Cu at (90.5, 84.2)
- added R83: 100k, Resistor_SMD:R_0603_1608Metric, F.Cu at (105.5, 74.9)
- added R84: 200k, Resistor_SMD:R_0603_1608Metric, F.Cu at (97.9, 74.9)
- added R85: 100k, Resistor_SMD:R_0603_1608Metric, F.Cu at (123.3, 60.4)
- added R86: 47k, Resistor_SMD:R_0603_1608Metric, F.Cu at (94.9, 76.4)
- added R87: 47k, Resistor_SMD:R_0603_1608Metric, F.Cu at (87.5, 84.2)
- added R88: 100k, Resistor_SMD:R_0603_1608Metric, F.Cu at (94.9, 74.9)
- added R89: 100k, Resistor_SMD:R_0603_1608Metric, F.Cu at (87.5, 85.8)
- added R9: 470, Resistor_SMD:R_0603_1608Metric, F.Cu at (162.3, 75.3)
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
Commit message: Added control switches.
Parts:
- added D10: 1N4148, Diode_THT:D_DO-35_SOD27_P7.62mm_Horizontal, F.Cu at (29.2, 50.3)
- added D11: 1N4148, Diode_THT:D_DO-35_SOD27_P7.62mm_Horizontal, F.Cu at (56.0, 41.5)
- added D12: 1N4148, Diode_THT:D_DO-35_SOD27_P7.62mm_Horizontal, F.Cu at (38.9, 50.3)
- added D13: 1N4148, Diode_THT:D_DO-35_SOD27_P7.62mm_Horizontal, F.Cu at (56.0, 36.4)
- added D14: 1N4148, Diode_THT:D_DO-35_SOD27_P7.62mm_Horizontal, F.Cu at (48.7, 50.3)
- added D15: 1N4148, Diode_THT:D_DO-35_SOD27_P7.62mm_Horizontal, F.Cu at (56.0, 38.9)
- added D5: LED, LED_THT:LED_D3.0mm, F.Cu at (38.7, 57.1)
- added D6: LED, LED_THT:LED_D3.0mm, F.Cu at (76.9, 31.2)
- added D7: LED, LED_THT:LED_D3.0mm, F.Cu at (50.1, 57.1)
- added D8: LM4040DBZ-10, Package_TO_SOT_SMD:SOT-23, F.Cu at (88.9, 23.0)
- added D9: 1N4148, Diode_THT:D_DO-35_SOD27_P7.62mm_Horizontal, F.Cu at (19.4, 50.3)
- added J4: Conn_01x03, Connector_PinHeader_2.54mm:PinHeader_1x03_P2.54mm_Vertical, F.Cu at (20.1, 56.6)
- added R100: 200k, Resistor_SMD:R_0603_1608Metric, F.Cu at (80.2, 25.0)
- added R101: 100k, Resistor_SMD:R_0603_1608Metric, F.Cu at (80.2, 23.5)
- added R102: 47k, Resistor_SMD:R_0603_1608Metric, F.Cu at (77.2, 25.0)
- added R103: 47k, Resistor_SMD:R_0603_1608Metric, F.Cu at (80.2, 21.9)
- added R104: 100k, Resistor_SMD:R_0603_1608Metric, F.Cu at (77.2, 23.5)
- added R105: 100k, Resistor_SMD:R_0603_1608Metric, F.Cu at (77.2, 21.9)
- added R106: 10k, Resistor_SMD:R_0603_1608Metric, F.Cu at (66.2, 35.8)
- added R107: 10k, Resistor_SMD:R_0603_1608Metric, F.Cu at (68.6, 23.5)
- added R108: 10k, Resistor_SMD:R_0603_1608Metric, F.Cu at (68.6, 21.9)
- added SW10: SW_SPDT_MSM, Local:SPDT, F.Cu at (36.6, 42.0)
- added SW11: SW_SPDT, Local:SPDT, F.Cu at (43.1, 25.0)
- added SW12: SW_SPDT, Local:SPDT, F.Cu at (61.0, 28.1)
- added SW6: SW_SPDT_MSM, Local:SPDT, F.Cu at (107.9, 64.4)
- added SW7: SW_SPDT_MSM, Local:SPDT, F.Cu at (128.2, 64.4)
- added SW8: SW_SPDT_MSM, Local:SPDT, F.Cu at (148.5, 64.4)
- added SW9: SW_SPDT_MSM, Local:SPDT, F.Cu at (168.8, 64.4)
- C1, C10, C11, C12, C13, C14, C15, C16, C17, C18, C19, C2, C20, C21, C22, C23, C24, C25, C26, C27, C28, C29, C3, C30, C31, C32, C33, C34, C35, C36, C37, C38, C39, C4, C40, C41, C42, C43, C44, C45, C46, C47, C48, C5, C6, C7, C8, C9, D1, D2, D3, Q1, Q2, Q3, Q4, R10, R19, R20, R23, R24, R43, R44, R45, R46, R5, R51, R52, R6, R65, R66, R7, R8, R83, R88, R89, R9, R95, R98, R99, U1, U10, U2, U3, U4, U5, U6, U7, U8, U9, X1: moved to B.Cu
- D4: value LM4040DBZ-10 -> LED; footprint Package_TO_SOT_SMD:SOT-23 -> LED_THT:LED_D3.0mm; moved to B.Cu
- J1: value Conn_02x05_Odd_Even -> Conn_02x03_Odd_Even; footprint Connector_PinHeader_2.54mm:PinHeader_2x05_P2.54mm_Vertical -> Connector_PinHeader_2.54mm:PinHeader_2x03_P2.54mm_Vertical; moved to B.Cu
- J2: value Conn_02x03_Odd_Even -> Conn_02x05_Odd_Even; footprint Connector_PinHeader_2.54mm:PinHeader_2x03_P2.54mm_Vertical -> Connector_PinHeader_2.54mm:PinHeader_2x05_P2.54mm_Vertical
- J3: value Conn_01x03 -> Conn_02x03_Odd_Even; footprint Connector_PinHeader_2.54mm:PinHeader_1x03_P2.54mm_Vertical -> Connector_PinHeader_2.54mm:PinHeader_2x03_P2.54mm_Vertical
- R1: value 330 -> 4k7; moved to B.Cu
- R11, R12, R47, R48: value 68k -> 470; moved to B.Cu
- R13, R14, R27, R28: value 33k -> 68k; moved to B.Cu
- R15, R16, R29, R30: value 68k -> 33k; moved to B.Cu
- R17, R55: value 470 -> 68k; moved to B.Cu
- R18, R56: value 1k5 -> 68k; moved to B.Cu
- R2: value 10k -> 4k7; moved to B.Cu
- R21, R57, R59: value 2k2 -> 470; moved to B.Cu
- R22, R58, R60: value 2k2 -> 1k5; moved to B.Cu
- R25, R26, R61, R62: value 68k -> 2k2; moved to B.Cu
- R3, R39, R41: value 470 -> 330; moved to B.Cu
- R31, R32: value 100k -> 68k; moved to B.Cu
- R33, R34, R37, R71, R72: value 1k -> 100k; moved to B.Cu
- R35, R73: value 100k -> 1k; moved to B.Cu
- R36, R74, R76, R78: value 10k -> 1k; moved to B.Cu
- R38: value 1k -> 10k; moved to B.Cu
- R4: value 470 -> 10k; moved to B.Cu
- R40, R42: value 470 -> 1k; moved to B.Cu
- R49, R50: value 33k -> 470; moved to B.Cu
- R53: value 470 -> 33k; moved to B.Cu
- R54: value 1k5 -> 33k; moved to B.Cu
- R63, R64: value 33k -> 2k2; moved to B.Cu
- R67, R68: value 100k -> 33k; moved to B.Cu
- R69, R70: value 1k -> 68k; moved to B.Cu
- R75, R77: value 100k -> 330; moved to B.Cu
- R79: value 2k2 -> 100k; moved to B.Cu
- R80, R82: value 100k -> 10k; moved to B.Cu
- R81, R91, R94: value 200k -> 100k; moved to B.Cu
- R84: value 200k -> 10k; moved to B.Cu
- R85: value 100k -> 2k2; moved to B.Cu
- R86, R96: value 47k -> 100k; moved to B.Cu
- R87, R97: value 47k -> 200k; moved to B.Cu
- R90: value 100k -> 200k; moved to B.Cu
- R92, R93: value 100k -> 47k; moved to B.Cu
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Connections:
- C37 pad 1: +12V -> +5V
- C38 pad 2: -12V -> GND
- C43 pad 1: +12V -> +5V
- C44 pad 2: -12V -> GND
- D4 pad 2: VRef-10 -> Net-(D4-Pad2)
- J1 pad 1: Net-(D2-Pad1) -> GND
- J1 pad 2: Net-(D2-Pad1) -> GND
- J1 pad 3: GND -> SDA
- J1 pad 4: GND -> SCL
- J1 pad 5: GND -> +5V
- J1 pad 6: GND -> +5V
- J2 pad 1: TRIG2 -> Net-(D2-Pad1)
- J2 pad 2: +5V -> Net-(D2-Pad1)
- J2 pad 3: TRIG3 -> GND
- J2 pad 4: TRIG1 -> GND
- J2 pad 5: Net-(J2-Pad5) -> GND
- J3 pad 1: GND -> TRIG2
- J3 pad 2: /MCU328/PD1-TXD -> +5V
- J3 pad 3: CV3 -> TRIG3
- R1 pad 2: Net-(D3-Pad2) -> SDA
- R10 pad 1: Net-(C16-Pad1) -> Net-(C14-Pad1)
- R10 pad 2: Net-(C14-Pad1) -> Net-(C12-Pad1)
- R11 pad 1: Net-(C17-Pad2) -> Net-(C15-Pad1)
- R11 pad 2: Net-(C15-Pad1) -> Net-(C13-Pad1)
- R12 pad 1: Net-(C18-Pad2) -> Net-(C16-Pad1)
- R12 pad 2: Net-(C16-Pad1) -> Net-(C14-Pad1)
- R13 pad 1: GND -> Net-(C17-Pad2)
- R13 pad 2: Net-(R13-Pad2) -> Net-(C15-Pad1)
- R14 pad 1: GND -> Net-(C18-Pad2)
- R14 pad 2: Net-(R14-Pad2) -> Net-(C16-Pad1)
- R15 pad 1: Net-(C17-Pad1) -> GND
- R15 pad 2: Net-(C17-Pad2) -> Net-(R15-Pad2)
- R16 pad 1: Net-(C18-Pad1) -> GND
- R16 pad 2: Net-(C18-Pad2) -> Net-(R16-Pad2)
- R17 pad 2: Net-(R17-Pad2) -> Net-(C17-Pad2)
- R18 pad 1: Net-(R18-Pad1) -> Net-(C18-Pad1)
- R18 pad 2: GND -> Net-(C18-Pad2)
- R19 pad 1: Net-(C18-Pad1) -> Net-(C17-Pad1)
- R2 pad 2: Net-(J2-Pad5) -> SCL
- R21 pad 1: Net-(C17-Pad1) -> Net-(C18-Pad1)
- R22 pad 1: Net-(R21-Pad2) -> Net-(R22-Pad1)
- R23 pad 1: Net-(C18-Pad1) -> Net-(C17-Pad1)
- R25 pad 1: Net-(R21-Pad2) -> Net-(C18-Pad1)
- R25 pad 2: Net-(C19-Pad2) -> Net-(R25-Pad2)
- R26 pad 1: Net-(R23-Pad2) -> Net-(R25-Pad2)
- R26 pad 2: Net-(C20-Pad2) -> GND
- R27 pad 1: GND -> Net-(R23-Pad2)
- R27 pad 2: Net-(R27-Pad2) -> Net-(C19-Pad2)
- R28 pad 1: GND -> Net-(R25-Pad2)
- R28 pad 2: Net-(R28-Pad2) -> Net-(C20-Pad2)
- R29 pad 1: Net-(C19-Pad1) -> GND
- R29 pad 2: Net-(C19-Pad2) -> Net-(R29-Pad2)
- R3 pad 1: Net-(C9-Pad1) -> +5V
- R3 pad 2: CV0 -> Net-(D3-Pad2)
- R30 pad 1: Net-(C20-Pad1) -> GND
- R30 pad 2: Net-(C20-Pad2) -> Net-(R30-Pad2)
- R31 pad 2: GND -> Net-(C19-Pad2)
- R32 pad 2: GND -> Net-(C20-Pad2)
- R33 pad 1: Net-(J-Inv1-PadT) -> Net-(C19-Pad1)
- R33 pad 2: Net-(C19-Pad1) -> GND
- R34 pad 1: Net-(J-Inv2-PadT) -> Net-(C20-Pad1)
- R34 pad 2: Net-(C20-Pad1) -> GND
- R35 pad 1: Net-(J-Inv3-PadT) -> Net-(J-Inv1-PadT)
- R35 pad 2: Net-(Q1-Pad1) -> Net-(C19-Pad1)
- R36 pad 1: +5V -> Net-(J-Inv2-PadT)
- R36 pad 2: CLK0 -> Net-(C20-Pad1)
- R37 pad 1: Net-(J-Inv4-PadT) -> Net-(J-Inv3-PadT)
- R37 pad 2: Net-(R37-Pad2) -> Net-(Q1-Pad1)
- R38 pad 1: Net-(J-Inv5-PadT) -> +5V
- R38 pad 2: Net-(R38-Pad2) -> CLK0
- R39 pad 1: Net-(C23-Pad1) -> TRIG0
- R39 pad 2: CV2 -> Net-(D4-Pad2)
- R4 pad 1: Net-(C10-Pad1) -> +5V
- R4 pad 2: CV1 -> Net-(J3-Pad5)
- R40 pad 1: Net-(C24-Pad1) -> Net-(J-Inv4-PadT)
- R40 pad 2: CV3 -> Net-(R40-Pad2)
- R41 pad 1: Net-(C25-Pad1) -> TRIG1
- R41 pad 2: Net-(C23-Pad1) -> Net-(D5-Pad2)
- R42 pad 1: Net-(C26-Pad1) -> Net-(J-Inv5-PadT)
- R42 pad 2: Net-(C24-Pad1) -> Net-(R42-Pad2)
- R43 pad 1: Net-(C27-Pad1) -> Net-(C23-Pad1)
- R43 pad 2: Net-(C25-Pad1) -> CV2
- R44 pad 1: Net-(C28-Pad1) -> Net-(C24-Pad1)
- R44 pad 2: Net-(C26-Pad1) -> CV3
- R45 pad 1: Net-(C29-Pad1) -> Net-(C25-Pad1)
- R45 pad 2: Net-(C27-Pad1) -> Net-(C23-Pad1)
- R46 pad 1: Net-(C30-Pad1) -> Net-(C26-Pad1)
- R46 pad 2: Net-(C28-Pad1) -> Net-(C24-Pad1)
- R47 pad 1: Net-(C31-Pad2) -> Net-(C27-Pad1)
- R47 pad 2: Net-(C29-Pad1) -> Net-(C25-Pad1)
- R48 pad 1: Net-(C32-Pad2) -> Net-(C28-Pad1)
- R48 pad 2: Net-(C30-Pad1) -> Net-(C26-Pad1)
- R49 pad 1: GND -> Net-(C29-Pad1)
- R49 pad 2: Net-(R49-Pad2) -> Net-(C27-Pad1)
- R5 pad 1: Net-(C11-Pad1) -> Net-(C9-Pad1)
- R5 pad 2: Net-(C9-Pad1) -> CV0
- R50 pad 1: GND -> Net-(C30-Pad1)
- R50 pad 2: Net-(R50-Pad2) -> Net-(C28-Pad1)
- R51 pad 1: Net-(C31-Pad1) -> Net-(C31-Pad2)
- R51 pad 2: Net-(C31-Pad2) -> Net-(C29-Pad1)
- R52 pad 1: Net-(C32-Pad1) -> Net-(C32-Pad2)
- R52 pad 2: Net-(C32-Pad2) -> Net-(C30-Pad1)
- R53 pad 1: Net-(C31-Pad1) -> GND
- R54 pad 1: Net-(R54-Pad1) -> GND
- R54 pad 2: GND -> Net-(R54-Pad2)
- R55 pad 1: Net-(C32-Pad1) -> Net-(C31-Pad1)
- R55 pad 2: Net-(R55-Pad2) -> Net-(C31-Pad2)
- R56 pad 1: Net-(R56-Pad1) -> Net-(C32-Pad1)
- R56 pad 2: GND -> Net-(C32-Pad2)
- R58 pad 1: Net-(R57-Pad2) -> Net-(R58-Pad1)
- R6 pad 1: Net-(C12-Pad1) -> Net-(C10-Pad1)
- R6 pad 2: Net-(C10-Pad1) -> CV1
- R60 pad 1: Net-(R59-Pad2) -> Net-(R60-Pad1)
- R61 pad 1: Net-(R57-Pad2) -> Net-(C31-Pad1)
- R61 pad 2: Net-(C33-Pad2) -> Net-(R61-Pad2)
- R62 pad 1: Net-(R59-Pad2) -> Net-(R61-Pad2)
- R62 pad 2: Net-(C34-Pad2) -> GND
- R63 pad 1: GND -> Net-(C32-Pad1)
- R64 pad 1: GND -> Net-(R63-Pad2)
- R64 pad 2: Net-(R64-Pad2) -> GND
- R65 pad 1: Net-(C33-Pad1) -> Net-(R61-Pad2)
- R66 pad 1: Net-(C34-Pad1) -> Net-(R63-Pad2)
- R67 pad 1: Net-(C33-Pad1) -> GND
- R67 pad 2: GND -> Net-(R67-Pad2)
- R68 pad 1: Net-(C34-Pad1) -> GND
- R68 pad 2: GND -> Net-(R68-Pad2)
- R69 pad 1: Net-(J-Inv6-PadT) -> Net-(C33-Pad1)
- R69 pad 2: Net-(C33-Pad1) -> Net-(C33-Pad2)
- R7 pad 1: Net-(C13-Pad1) -> Net-(C11-Pad1)
- R7 pad 2: Net-(C11-Pad1) -> Net-(C9-Pad1)
- R70 pad 1: Net-(J-Inv7-PadT) -> Net-(C34-Pad1)
- R70 pad 2: Net-(C34-Pad1) -> Net-(C34-Pad2)
- R71 pad 1: Net-(J-Inv8-PadT) -> Net-(C33-Pad1)
- R71 pad 2: Net-(R71-Pad2) -> GND
- R72 pad 1: Net-(J-Inv9-PadT) -> Net-(C34-Pad1)
- R72 pad 2: Net-(R72-Pad2) -> GND
- R73 pad 1: Net-(J-Inv10-PadT) -> Net-(J-Inv6-PadT)
- R73 pad 2: Net-(Q2-Pad1) -> Net-(C33-Pad1)
- R74 pad 1: +5V -> Net-(J-Inv7-PadT)
- R74 pad 2: RST0 -> Net-(C34-Pad1)
- R75 pad 1: Net-(J-Inv11-PadT) -> TRIG2
- R75 pad 2: Net-(Q3-Pad1) -> Net-(D6-Pad2)
- R76 pad 1: +5V -> Net-(J-Inv8-PadT)
- R76 pad 2: CLK1 -> Net-(R76-Pad2)
- R77 pad 1: Net-(J-Inv12-PadT) -> TRIG3
- R77 pad 2: Net-(Q4-Pad1) -> Net-(D7-Pad2)
- R78 pad 1: +5V -> Net-(J-Inv9-PadT)
- R78 pad 2: RST1 -> Net-(R78-Pad2)
- R79 pad 1: -12V -> Net-(J-Inv10-PadT)
- R79 pad 2: VRef-10 -> Net-(Q2-Pad1)
- R8 pad 1: Net-(C14-Pad1) -> Net-(C12-Pad1)
- R8 pad 2: Net-(C12-Pad1) -> Net-(C10-Pad1)
- R80 pad 1: Net-(R80-Pad1) -> +5V
- R80 pad 2: Net-(C41-Pad2) -> RST0
- R81 pad 1: VRef-10 -> Net-(J-Inv11-PadT)
- R81 pad 2: Net-(C41-Pad2) -> Net-(Q3-Pad1)
- R82 pad 1: Net-(J-Inv13-PadT) -> +5V
- R82 pad 2: Net-(C41-Pad2) -> CLK1
- R83 pad 1: Net-(R83-Pad1) -> Net-(J-Inv12-PadT)
- R83 pad 2: Net-(C42-Pad2) -> Net-(Q4-Pad1)
- R84 pad 1: VRef-10 -> +5V
- R84 pad 2: Net-(C42-Pad2) -> RST1
- R85 pad 1: Net-(J-Inv14-PadT) -> -12V
- R85 pad 2: Net-(C42-Pad2) -> VRef-10
- R86 pad 2: GND -> Net-(C41-Pad2)
- R87 pad 1: Net-(R87-Pad1) -> VRef-10
- R87 pad 2: GND -> Net-(C41-Pad2)
- R88 pad 1: STA0 -> Net-(J-Inv13-PadT)
- R89 pad 1: END0 -> Net-(R89-Pad1)
- R9 pad 1: Net-(C15-Pad1) -> Net-(C13-Pad1)
- R9 pad 2: Net-(C13-Pad1) -> Net-(C11-Pad1)
- R90 pad 1: Net-(R90-Pad1) -> VRef-10
- R90 pad 2: Net-(C47-Pad2) -> Net-(C42-Pad2)
- R91 pad 1: VRef-10 -> Net-(J-Inv14-PadT)
- R91 pad 2: Net-(C47-Pad2) -> Net-(C42-Pad2)
- R92 pad 1: Net-(J-Inv15-PadT) -> Net-(R92-Pad1)
- R92 pad 2: Net-(C47-Pad2) -> GND
- R93 pad 2: Net-(C48-Pad2) -> GND
- R94 pad 1: VRef-10 -> STA0
- R94 pad 2: Net-(C48-Pad2) -> Net-(C41-Pad2)
- R95 pad 1: Net-(J-Inv16-PadT) -> END0
- R95 pad 2: Net-(C48-Pad2) -> Net-(C42-Pad2)
- R96 pad 2: GND -> Net-(C47-Pad2)
- R97 pad 1: Net-(R97-Pad1) -> VRef-10
- R97 pad 2: GND -> Net-(C47-Pad2)
- R98 pad 1: STA1 -> Net-(J-Inv15-PadT)
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Other:
- board outline added: 100.6 x 100 mm

Commit message: Inital placement.
Parts:
- added C49: 47n, Capacitor_SMD:C_0603_1608Metric, B.Cu at (178.9, 101.5)
- added C50: 47n, Capacitor_SMD:C_0603_1608Metric, B.Cu at (175.9, 106.0)
- added C51: 100p, Capacitor_SMD:C_0603_1608Metric, B.Cu at (178.4, 112.5)
- added C52: 100p, Capacitor_SMD:C_0603_1608Metric, B.Cu at (182.4, 109.8)
- added U11: 74AHCT1G125, Package_TO_SOT_SMD:SOT-23-5, B.Cu at (189.0, 139.5)
- added U12: TL072, Package_SO:MSOP-8_3x3mm_P0.65mm, B.Cu at (157.6, 107.8)
- added U13: 74AHCT1G125, Package_TO_SOT_SMD:SOT-23-5, B.Cu at (188.8, 149.0)
- added U14: TL072, Package_SO:MSOP-8_3x3mm_P0.65mm, B.Cu at (177.7, 108.6)
- C10, C12, C13, C15, C16, C29, C30, C9: value 47n -> 100n
- C11, C14: value 47n -> 470p
- C17, C20: value 100p -> 470p
- C18, C19: value 100p -> 100n
- C27, C28: value 47n -> 100p
- C31, C32, C33, C34: value 100p -> 47n
- C35, C36, C43, C44: value 100n -> 100p
- C39, C40: value 100n -> 47n
- C41, C42, C47, C48: value 470p -> 47n
- D10, D11, D12, D9: footprint Diode_THT:D_DO-35_SOD27_P7.62mm_Horizontal -> Diode_SMD:D_SOD-123; moved to B.Cu
- D13, D14, D15: value 1N4148 -> LED; footprint Diode_THT:D_DO-35_SOD27_P7.62mm_Horizontal -> LED_THT:LED_D3.0mm
- D4: moved to F.Cu
- D5: value LED -> LM4040DBZ-10; footprint LED_THT:LED_D3.0mm -> Package_TO_SOT_SMD:SOT-23; moved to B.Cu
- D6, D7: value LED -> 1N4148; footprint LED_THT:LED_D3.0mm -> Diode_SMD:D_SOD-123; moved to B.Cu
- D8: value LM4040DBZ-10 -> 1N4148; footprint Package_TO_SOT_SMD:SOT-23 -> Diode_SMD:D_SOD-123; moved to B.Cu
- J2, J3, J4: moved to B.Cu
- R10, R12, R21, R8: value 470 -> 100k
- R100: value 200k -> 470; moved to B.Cu
- R101: value 100k -> 1k5; moved to B.Cu
- R102, R103: value 47k -> 2k2; moved to B.Cu
- R104: value 100k -> 68k; moved to B.Cu
- R105: value 100k -> 33k; moved to B.Cu
- R106: value 10k -> 68k; moved to B.Cu
- R107: value 10k -> 100k; moved to B.Cu
- R108: value 10k -> 1k; moved to B.Cu
- R11, R19: value 470 -> 47k
- R13, R14, R32: value 68k -> 10k
- R15: value 33k -> 10k
- R16, R30, R53: value 33k -> 100k
- R17, R27: value 68k -> 200k
- R18, R28, R31: value 68k -> 100k
- R20: value 1k5 -> 100k
- R22: value 1k5 -> 200k
- R23, R25, R26: value 2k2 -> 100k
- R24: value 2k2 -> 47k
- R29: value 33k -> 47k
- R34: value 100k -> 10k
- R35: value 1k -> 100k
- R36: value 1k -> 10k
- R39, R41, R75, R77: value 330 -> 470
- R40, R42, R76, R78: value 1k -> 470
- R43, R45, R50: value 470 -> 68k
- R44: value 470 -> 33k
- R47: value 470 -> 1k5
- R48, R49, R7: value 470 -> 2k2
- R5: value 470 -> 330
- R51, R69: value 68k -> 33k
- R54: value 33k -> 1k
- R55: value 68k -> 330
- R56: value 68k -> 1k
- R58, R60: value 1k5 -> 470
- R6: value 470 -> 1k
- R61, R63: value 2k2 -> 68k
- R62: value 2k2 -> 33k
- R64: value 2k2 -> 470
- R65: value 68k -> 1k5
- R66: value 68k -> 2k2
- R67: value 33k -> 2k2
- R68: value 33k -> 68k
- R72: value 100k -> 1k
- R73: value 1k -> 330
- R79, R81, R86, R88, R99: value 100k -> 68k
- R80: value 10k -> 33k
- R82: value 10k -> 470
- R83: value 100k -> 1k5
- R84: value 10k -> 2k2
- R87: value 200k -> 33k
- R9: value 470 -> 200k
- R90: value 200k -> 1k
- R91: value 100k -> 330
- R92: value 47k -> 1k
- R93: value 47k -> 470
- R94, R95, R96: value 100k -> 470
- R97: value 200k -> 68k
- R98: value 100k -> 33k
- SW11, SW12: value SW_SPDT -> SW_SPDT_MSM
- SW7, SW8: value SW_SPDT_MSM -> SW_SPDT
- U1: footprint Package_TO_SOT_THT:TO-220-3_Vertical -> Package_TO_SOT_SMD:TO-252-3_TabPin2
- U10: value MCP6004 -> TL072; footprint Package_SO:SOIC-14_3.9x8.7mm_P1.27mm -> Package_SO:MSOP-8_3x3mm_P0.65mm
- U3: value TL074 -> 74AHCT1G125; footprint Package_SO:SOIC-14_3.9x8.7mm_P1.27mm -> Package_TO_SOT_SMD:SOT-23-5
- U4, U5, U7: value 74AHCT1G125 -> MCP6002-xMS; footprint Package_TO_SOT_SMD:SOT-23-5 -> Package_SO:MSOP-8_3x3mm_P0.65mm
- U6: value TL074 -> MCP6002-xMS; footprint Package_SO:SOIC-14_3.9x8.7mm_P1.27mm -> Package_SO:MSOP-8_3x3mm_P0.65mm
- U8: value 74AHCT1G125 -> TL072; footprint Package_TO_SOT_SMD:SOT-23-5 -> Package_SO:MSOP-8_3x3mm_P0.65mm
- U9: value MCP6004 -> 74AHCT1G125; footprint Package_SO:SOIC-14_3.9x8.7mm_P1.27mm -> Package_TO_SOT_SMD:SOT-23-5
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Connections:
- C11 pad 1: Net-(C11-Pad1) -> STA0
- C11 pad 2: GND -> Net-(C11-Pad2)
- C12 pad 1: Net-(C12-Pad1) -> +5V
- C14 pad 1: Net-(C14-Pad1) -> END0
- C14 pad 2: GND -> Net-(C14-Pad2)
- C15 pad 1: Net-(C15-Pad1) -> +5V
- C17 pad 1: Net-(C17-Pad1) -> STA1
- C18 pad 1: Net-(C18-Pad1) -> +5V
- C18 pad 2: Net-(C18-Pad2) -> GND
- C19 pad 2: Net-(C19-Pad2) -> GND
- C20 pad 1: Net-(C20-Pad1) -> END1
- C27 pad 2: GND -> Net-(C27-Pad2)
- C28 pad 2: GND -> Net-(C28-Pad2)
- C29 pad 1: Net-(C29-Pad1) -> +12V
- C30 pad 1: Net-(C30-Pad1) -> GND
- C30 pad 2: GND -> -12V
- C31 pad 2: Net-(C31-Pad2) -> GND
- C32 pad 2: Net-(C32-Pad2) -> GND
- C33 pad 2: Net-(C33-Pad2) -> GND
- C34 pad 2: Net-(C34-Pad2) -> GND
- C35 pad 1: +12V -> Net-(C35-Pad1)
- C35 pad 2: GND -> Net-(C35-Pad2)
- C36 pad 1: GND -> Net-(C36-Pad1)
- C36 pad 2: -12V -> Net-(C36-Pad2)
- C37 pad 1: +5V -> +12V
- C38 pad 2: GND -> -12V
- C41 pad 1: STA0 -> Net-(C41-Pad1)
- C41 pad 2: Net-(C41-Pad2) -> GND
- C42 pad 1: END0 -> Net-(C42-Pad1)
- C42 pad 2: Net-(C42-Pad2) -> GND
- C43 pad 1: +5V -> Net-(C43-Pad1)
- C43 pad 2: GND -> Net-(C43-Pad2)
- C44 pad 1: GND -> Net-(C44-Pad1)
- C44 pad 2: GND -> Net-(C44-Pad2)
- C45 pad 1: Net-(C45-Pad1) -> +12V
- C46 pad 1: Net-(C46-Pad1) -> GND
- C46 pad 2: GND -> -12V
- C47 pad 1: STA1 -> Net-(C47-Pad1)
- C47 pad 2: Net-(C47-Pad2) -> GND
- C48 pad 1: END1 -> Net-(C48-Pad1)
- C48 pad 2: Net-(C48-Pad2) -> GND
- C9 pad 1: Net-(C9-Pad1) -> +5V
- D10 pad 1: Scan1 -> Net-(D10-Pad1)
- D10 pad 2: Net-(D10-Pad2) -> Sense2
- D11 pad 1: Scan2 -> Net-(D11-Pad1)
- D11 pad 2: Net-(D11-Pad2) -> Sense2
- D12 pad 1: Scan3 -> Net-(D12-Pad1)
- D12 pad 2: Net-(D12-Pad2) -> Sense2
- D13 pad 1: Net-(D13-Pad1) -> GND
- D13 pad 2: Sense2 -> Net-(D13-Pad2)
- D14 pad 1: Net-(D14-Pad1) -> GND
- D14 pad 2: Sense2 -> Net-(D14-Pad2)
- D15 pad 1: Net-(D15-Pad1) -> GND
- D15 pad 2: Sense2 -> Net-(D15-Pad2)
- D5 pad 2: Net-(D5-Pad2) -> VRef-10
- D6 pad 1: GND -> Scan0
- D7 pad 1: GND -> Scan1
- D8 pad 1: GND -> Scan2
- D8 pad 2: VRef-10 -> Net-(D8-Pad2)
- D9 pad 1: Scan0 -> Scan3
- J-Inv1 pad T: Net-(J-Inv1-PadT) -> /DigitalIn/In
- J-Inv1 pad TN: Net-(J-Inv1-PadTN) -> +5V
- J-Inv10 pad T: Net-(J-Inv10-PadT) -> /DigitalOut/Out
- J-Inv10 pad TN: GND -> Net-(J-Inv10-PadTN)
- J-Inv11 pad T: Net-(J-Inv11-PadT) -> /sheet5C230BC3/Out
- J-Inv11 pad TN: CLK0 -> Net-(J-Inv11-PadTN)
- J-Inv12 pad T: Net-(J-Inv12-PadT) -> /sheet5C230BAE/Out
- J-Inv12 pad TN: RST0 -> Net-(J-Inv12-PadTN)
- J-Inv13 pad T: Net-(J-Inv13-PadT) -> /sheet5C25BE7D/Out
- J-Inv13 pad TN: GND -> Net-(J-Inv13-PadTN)
- J-Inv14 pad T: Net-(J-Inv14-PadT) -> /sheet5C25BE68/Out
- J-Inv14 pad TN: Net-(J-Inv13-PadT) -> Net-(J-Inv14-PadTN)
- J-Inv15 pad T: Net-(J-Inv15-PadT) -> /sheet5C25BEB7/Out
- J-Inv15 pad TN: GND -> Net-(J-Inv15-PadTN)
- J-Inv16 pad T: Net-(J-Inv16-PadT) -> /sheet5C25BE94/Out
- J-Inv16 pad TN: Net-(J-Inv15-PadT) -> Net-(J-Inv16-PadTN)
- J-Inv2 pad T: Net-(J-Inv2-PadT) -> /sheet5C188821/In
- J-Inv2 pad TN: Net-(J-Inv2-PadTN) -> GND
- J-Inv3 pad T: Net-(J-Inv3-PadT) -> /sheet5C192077/In
- J-Inv3 pad TN: +5V -> /DigitalIn/In
- J-Inv4 pad T: Net-(J-Inv4-PadT) -> /sheet5C19208D/In
- J-Inv4 pad TN: Net-(J-Inv4-PadTN) -> /sheet5C188821/In
- J-Inv5 pad T: Net-(J-Inv5-PadT) -> /CVIn/In
- J-Inv5 pad TN: Net-(J-Inv5-PadTN) -> GND
- J-Inv6 pad T: Net-(J-Inv6-PadT) -> /sheet5C14AC01/In
- J-Inv6 pad TN: Net-(J-Inv6-PadTN) -> /CVIn/In
- J-Inv7 pad T: Net-(J-Inv7-PadT) -> /sheet5C1536C4/In
- J-Inv7 pad TN: Net-(J-Inv7-PadTN) -> /CVIn/In
- J-Inv8 pad T: Net-(J-Inv8-PadT) -> /sheet5C1536DC/In
- J-Inv8 pad TN: Net-(J-Inv8-PadTN) -> /sheet5C1536C4/In
- J-Inv9 pad T: Net-(J-Inv9-PadT) -> /CVOut/Out
- R10 pad 1: Net-(C14-Pad1) -> /CVIn/In
- R10 pad 2: Net-(C12-Pad1) -> Net-(C11-Pad2)
- R100 pad 1: VRef-10 -> Net-(C51-Pad1)
- R100 pad 2: Net-(C48-Pad2) -> Net-(R100-Pad2)
- R101 pad 1: Net-(J-Inv16-PadT) -> Net-(R101-Pad1)
- R101 pad 2: Net-(C48-Pad2) -> GND
- R102 pad 1: Net-(R102-Pad1) -> Net-(C51-Pad1)
- R102 pad 2: GND -> Net-(R102-Pad2)
- R103 pad 1: Net-(R103-Pad1) -> Net-(R102-Pad2)
- R104 pad 1: STA1 -> Net-(R102-Pad2)
- R104 pad 2: Net-(C47-Pad2) -> Net-(C52-Pad2)
- R105 pad 1: END1 -> GND
- R105 pad 2: Net-(C48-Pad2) -> Net-(R105-Pad2)
- R106 pad 1: +5V -> Net-(C52-Pad1)
- R106 pad 2: Sense0 -> Net-(C52-Pad2)
- R107 pad 1: +5V -> Net-(C52-Pad1)
- R107 pad 2: Sense1 -> GND
- R108 pad 1: +5V -> /sheet5C25BEB7/Out
- R108 pad 2: Sense2 -> Net-(C52-Pad1)
- R11 pad 1: Net-(C15-Pad1) -> Net-(R11-Pad1)
- R11 pad 2: Net-(C13-Pad1) -> GND
- R12 pad 1: Net-(C16-Pad1) -> STA0
- R12 pad 2: Net-(C14-Pad1) -> Net-(C11-Pad2)
- R13 pad 1: Net-(C17-Pad2) -> +5V
- R13 pad 2: Net-(C15-Pad1) -> Sense0
- R14 pad 1: Net-(C18-Pad2) -> +5V
- R14 pad 2: Net-(C16-Pad1) -> Sense1
- R15 pad 1: GND -> +5V
- R15 pad 2: Net-(R15-Pad2) -> Sense2
- R16 pad 1: GND -> Net-(R16-Pad1)
- R16 pad 2: Net-(R16-Pad2) -> Net-(C14-Pad2)
- R17 pad 1: Net-(C17-Pad1) -> VRef-10
- R17 pad 2: Net-(C17-Pad2) -> Net-(C14-Pad2)
- R18 pad 1: Net-(C18-Pad1) -> /sheet5C14AC01/In
- R18 pad 2: Net-(C18-Pad2) -> Net-(C14-Pad2)
- R19 pad 1: Net-(C17-Pad1) -> Net-(R19-Pad1)
- R19 pad 2: Net-(R19-Pad2) -> GND
- R20 pad 1: Net-(R20-Pad1) -> END0
- R20 pad 2: GND -> Net-(C14-Pad2)
- R21 pad 1: Net-(C18-Pad1) -> Net-(R21-Pad1)
- R21 pad 2: Net-(R21-Pad2) -> Net-(C17-Pad2)
- R22 pad 1: Net-(R22-Pad1) -> VRef-10
- R22 pad 2: GND -> Net-(C17-Pad2)
- R23 pad 1: Net-(C17-Pad1) -> /sheet5C1536C4/In
- R23 pad 2: Net-(R23-Pad2) -> Net-(C17-Pad2)
- R24 pad 1: Net-(R23-Pad2) -> Net-(R24-Pad1)
- R25 pad 1: Net-(C18-Pad1) -> STA1
- R25 pad 2: Net-(R25-Pad2) -> Net-(C17-Pad2)
- R26 pad 1: Net-(R25-Pad2) -> Net-(R26-Pad1)
- R26 pad 2: GND -> Net-(C20-Pad2)
- R27 pad 1: Net-(R23-Pad2) -> VRef-10
- R27 pad 2: Net-(C19-Pad2) -> Net-(C20-Pad2)
- R28 pad 1: Net-(R25-Pad2) -> /sheet5C1536DC/In
- R29 pad 1: GND -> Net-(R29-Pad1)
- R29 pad 2: Net-(R29-Pad2) -> GND
- R30 pad 1: GND -> END1
- R30 pad 2: Net-(R30-Pad2) -> Net-(C20-Pad2)
- R31 pad 1: Net-(C19-Pad1) -> /DigitalIn/In
- R31 pad 2: Net-(C19-Pad2) -> Net-(Q1-Pad1)
- R32 pad 1: Net-(C20-Pad1) -> +5V
- R32 pad 2: Net-(C20-Pad2) -> CLK0
- R33 pad 1: Net-(C19-Pad1) -> /sheet5C188821/In
- R33 pad 2: GND -> Net-(Q2-Pad1)
- R34 pad 1: Net-(C20-Pad1) -> +5V
- R34 pad 2: GND -> RST0
- R35 pad 1: Net-(J-Inv1-PadT) -> /sheet5C192077/In
- R35 pad 2: Net-(C19-Pad1) -> Net-(Q3-Pad1)
- R36 pad 1: Net-(J-Inv2-PadT) -> +5V
- R36 pad 2: Net-(C20-Pad1) -> CLK1
- R37 pad 1: Net-(J-Inv3-PadT) -> /sheet5C19208D/In
- R37 pad 2: Net-(Q1-Pad1) -> Net-(Q4-Pad1)
- R38 pad 2: CLK0 -> RST1
- R39 pad 1: TRIG0 -> Net-(C23-Pad1)
- R39 pad 2: Net-(D4-Pad2) -> CV0
- R40 pad 1: Net-(J-Inv4-PadT) -> Net-(C24-Pad1)
- R40 pad 2: Net-(R40-Pad2) -> Net-(C23-Pad1)
- R41 pad 1: TRIG1 -> Net-(C25-Pad1)
- R41 pad 2: Net-(D5-Pad2) -> Net-(C24-Pad1)
- R42 pad 1: Net-(J-Inv5-PadT) -> Net-(C26-Pad1)
- R42 pad 2: Net-(R42-Pad2) -> Net-(C25-Pad1)
- R43 pad 1: Net-(C23-Pad1) -> Net-(C27-Pad2)
- R43 pad 2: CV2 -> Net-(C26-Pad1)
- R44 pad 1: Net-(C24-Pad1) -> GND
- R44 pad 2: CV3 -> Net-(R44-Pad2)
- R45 pad 1: Net-(C25-Pad1) -> Net-(C27-Pad1)
- R45 pad 2: Net-(C23-Pad1) -> Net-(C27-Pad2)
- R46 pad 1: Net-(C26-Pad1) -> Net-(C27-Pad1)
- R46 pad 2: Net-(C24-Pad1) -> Net-(R46-Pad2)
- R47 pad 1: Net-(C27-Pad1) -> Net-(R47-Pad1)
- R47 pad 2: Net-(C25-Pad1) -> GND
- R48 pad 1: Net-(C28-Pad1) -> Net-(C27-Pad1)
- R48 pad 2: Net-(C26-Pad1) -> Net-(R48-Pad2)
- R49 pad 1: Net-(C29-Pad1) -> Net-(R48-Pad2)
- R49 pad 2: Net-(C27-Pad1) -> GND
- R5 pad 1: Net-(C9-Pad1) -> TRIG0
- R5 pad 2: CV0 -> Net-(D4-Pad2)
- R50 pad 1: Net-(C30-Pad1) -> Net-(R48-Pad2)
- R50 pad 2: Net-(C28-Pad1) -> Net-(C28-Pad2)
- R51 pad 1: Net-(C31-Pad2) -> GND
- R51 pad 2: Net-(C29-Pad1) -> Net-(R51-Pad2)
- R52 pad 1: Net-(C32-Pad2) -> Net-(C28-Pad1)
- R52 pad 2: Net-(C30-Pad1) -> Net-(C28-Pad2)
- R53 pad 1: GND -> Net-(C28-Pad1)
- R53 pad 2: Net-(R53-Pad2) -> GND
- R54 pad 1: GND -> /CVOut/Out
- R54 pad 2: Net-(R54-Pad2) -> Net-(C28-Pad1)
- R55 pad 1: Net-(C31-Pad1) -> TRIG1
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
Commit message: More layout.
Parts:
- moved R54 41.0 mm to (107.9, 138.0)
- moved R47 20.4 mm to (100.2, 107.5)
- moved R49 18.7 mm to (100.2, 105.0)
- moved R48 17.9 mm to (122.7, 112.4), turned to 90 degrees
- moved C25 17.0 mm to (114.2, 95.8), turned to 270 degrees
- moved R40 16.3 mm to (119.2, 95.8)
- moved C26 14.9 mm to (114.2, 92.0), turned to 270 degrees
- moved R46 14.9 mm to (100.2, 102.5)
- moved C23 13.7 mm to (121.8, 92.0), turned to 90 degrees
- moved R52 12.7 mm to (122.7, 99.7), turned to 270 degrees
- moved R51 12.0 mm to (117.6, 99.7), turned to 270 degrees
- moved R42 11.8 mm to (116.7, 92.0), turned to 270 degrees
- moved C24 9.28 mm to (121.8, 95.8), turned to 90 degrees
- moved R44 9.06 mm to (117.6, 112.4), turned to 90 degrees
- moved R39 8.88 mm to (119.2, 92.0), turned to 90 degrees
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Connections:
- C1 pad 2: GND -> (no net)
- C10 pad 2: GND -> (no net)
- C12 pad 2: GND -> (no net)
- C13 pad 2: GND -> (no net)
- C15 pad 2: GND -> (no net)
- C16 pad 2: GND -> (no net)
- C18 pad 2: GND -> (no net)
- C19 pad 2: GND -> (no net)
- C2 pad 1: GND -> (no net)
- C21 pad 2: GND -> (no net)
- C22 pad 1: GND -> (no net)
- C23 pad 2: GND -> (no net)
- C24 pad 2: GND -> (no net)
- C25 pad 2: GND -> (no net)
- C26 pad 2: GND -> (no net)
- C29 pad 2: GND -> (no net)
- C3 pad 2: GND -> (no net)
- C30 pad 1: GND -> (no net)
- C31 pad 2: GND -> (no net)
- C32 pad 2: GND -> (no net)
- C33 pad 2: GND -> (no net)
- C34 pad 2: GND -> (no net)
- C37 pad 2: GND -> (no net)
- C38 pad 1: GND -> (no net)
- C39 pad 2: GND -> (no net)
- C4 pad 2: GND -> (no net)
- C40 pad 2: GND -> (no net)
- C41 pad 2: GND -> (no net)
- C42 pad 2: GND -> (no net)
- C45 pad 2: GND -> (no net)
- C46 pad 1: GND -> (no net)
- C47 pad 2: GND -> (no net)
- C48 pad 2: GND -> (no net)
- C49 pad 2: GND -> (no net)
- C5 pad 2: GND -> (no net)
- C50 pad 2: GND -> (no net)
- C6 pad 1: GND -> (no net)
- C7 pad 2: GND -> (no net)
- C8 pad 1: GND -> (no net)
- C9 pad 2: GND -> (no net)
- D13 pad 1: GND -> (no net)
- D14 pad 1: GND -> (no net)
- D15 pad 1: GND -> (no net)
- D3 pad 1: GND -> (no net)
- D4 pad 1: GND -> (no net)
- D5 pad 1: GND -> (no net)
- J-Inv1 pad S: GND -> (no net)
- J-Inv10 pad S: GND -> (no net)
- J-Inv11 pad S: GND -> (no net)
- J-Inv12 pad S: GND -> (no net)
- J-Inv13 pad S: GND -> (no net)
- J-Inv14 pad S: GND -> (no net)
- J-Inv15 pad S: GND -> (no net)
- J-Inv16 pad S: GND -> (no net)
- J-Inv2 pad S: GND -> (no net)
- J-Inv2 pad TN: GND -> (no net)
- J-Inv3 pad S: GND -> (no net)
- J-Inv4 pad S: GND -> (no net)
- J-Inv5 pad S: GND -> (no net)
- J-Inv5 pad TN: GND -> (no net)
- J-Inv6 pad S: GND -> (no net)
- J-Inv7 pad S: GND -> (no net)
- J-Inv8 pad S: GND -> (no net)
- J-Inv9 pad S: GND -> (no net)
- J1 pad 1: GND -> (no net)
- J1 pad 2: GND -> (no net)
- J2 pad 3: GND -> (no net)
- J2 pad 4: GND -> (no net)
- J2 pad 5: GND -> (no net)
- J2 pad 6: GND -> (no net)
- J2 pad 7: GND -> (no net)
- J2 pad 8: GND -> (no net)
- J3 pad 6: GND -> (no net)
- J4 pad 1: GND -> (no net)
- Q1 pad 2: GND -> (no net)
- Q2 pad 2: GND -> (no net)
- Q3 pad 2: GND -> (no net)
- Q4 pad 2: GND -> (no net)
- R101 pad 2: GND -> (no net)
- R103 pad 2: GND -> (no net)
- R105 pad 1: GND -> (no net)
- R107 pad 2: GND -> (no net)
- R11 pad 2: GND -> (no net)
- R19 pad 2: GND -> (no net)
- R24 pad 2: GND -> (no net)
- R29 pad 2: GND -> (no net)
- R44 pad 1: GND -> (no net)
- R47 pad 2: GND -> (no net)
- R49 pad 2: GND -> (no net)
- R51 pad 1: GND -> (no net)
- R53 pad 2: GND -> (no net)
- R62 pad 1: GND -> (no net)
- R65 pad 2: GND -> (no net)
- R67 pad 2: GND -> (no net)
- R69 pad 1: GND -> (no net)
- R71 pad 2: GND -> (no net)
- R80 pad 1: GND -> (no net)
- R83 pad 2: GND -> (no net)
- R85 pad 2: GND -> (no net)
- R87 pad 1: GND -> (no net)
- R89 pad 2: GND -> (no net)
- R98 pad 1: GND -> (no net)
- RV1 pad 3: GND -> (no net)
- RV2 pad 3: GND -> (no net)
- RV3 pad 3: GND -> (no net)
- RV4 pad 3: GND -> (no net)
- SW1 pad 2: GND -> (no net)
- U1 pad 2: GND -> (no net)
- U11 pad 1: GND -> (no net)
- U11 pad 3: GND -> (no net)
- U13 pad 1: GND -> (no net)
- U13 pad 3: GND -> (no net)
- U2 pad 21: GND -> (no net)
- U2 pad 5: GND -> (no net)
- U3 pad 1: GND -> (no net)
- U3 pad 3: GND -> (no net)
- U4 pad 4: GND -> (no net)
- U5 pad 4: GND -> (no net)
- U6 pad 4: GND -> (no net)
- U7 pad 4: GND -> (no net)
- U9 pad 1: GND -> (no net)
- U9 pad 3: GND -> (no net)
- X1 pad 2: GND -> (no net)
